Commit message: ♥ usb캠에서 tf 반대로 표출되는 문제 수정

File: tetraDS_description/urdf/tetraDS/tetraDS.xacro (robot description, xacro)
@@ -70,5 +70,5 @@
   </link>
   <joint name="usb_cam" type="fixed">
-    <origin xyz="0.135 0.0 0.181" rpy="1.5708 3.14159 4.71239"/>
+    <origin xyz="0.135 0.0 0.181" rpy="1.5708 3.14159 1.5708"/>
     <parent link="base_link"/>
     <child link="usb_cam" />

Commit message: ♥ 카메라 2로 기입된것을 1으로 변경

File: tetraDS_description/urdf/tetraDS/tetraDS.xacro (robot description, xacro)
@@ -88,6 +88,5 @@
     <child link="Front_bumper" />
   </joint>
-<!-- 240314 mwcha Removed 'camera1_link' because S model just have a single depth camera -->
-   <link name="camera2_link">
+   <link name="camera1_link">
       <visual>
         <origin xyz="0 0 0" rpy="0 0 0" />
@@ -98,9 +97,9 @@
       </visual>
   </link>
-  <joint name="camera2_link" type="fixed">
+  <joint name="camera1_link" type="fixed">
     <!--<origin xyz="0.1553 -0.1155 0.0" rpy="3.14 -0.261799 0" />-->
     <origin xyz="0.1347 0.0 0.1344" rpy="0 0 0" />
     <parent link="base_link"/>
-    <child link="camera2_link" />
+    <child link="camera1_link" />
   </joint>
  <link name="base_Upperlink">
